Commit message: Add Gemini 305 wrist camera setup and domain randomization
- Configure TiledCamera with Gemini 305 depth intrinsics (80x50, 88° HFOV,
  focal_length=3.19mm, depth range 4-100cm) as default in base.yaml
- Move old Kuka camera values to kuka_allegro robot layer
- Fix URDF optical frame rotation (rpy 0,0,π instead of -π/2,0,-π/2)
- Change WristCameraConfig from single resolution to width + height
- Add robot base position domain randomization (±1cm XY, 5mm-2cm Z)
- Add camera offset domain randomization (±2mm, camera-frame perturbation)
- New reset_camera_offset event function in mdp/events.py
- Add base_plate mesh visual to URDF

Co-Authored-By: Claude Opus 4.6 <noreply@anthropic.com>

File: source/isaaclab_tasks/isaaclab_tasks/manager_based/manipulation/y2r/assets/ur5e_leap/ur5e_leap_right_gemini305.urdf (robot description, URDF)
Before this commit: robot ur5e_leap_right, 40 links, 39 joints
Links:
- link base: geometry visual mesh filename=meshes/base_plate.obj
Joints:
- joint gemini_305_left_optical_joint: origin xyz=0 0 0 rpy=-1.5707963 0 -1.5707963 -> xyz=0 0 0 rpy=0 0 3.14159265
- joint gemini_305_right_optical_joint: origin xyz=0 0 0 rpy=-1.5707963 0 -1.5707963 -> xyz=0 0 0 rpy=0 0 3.14159265

Commit message: Simplify collision geometry for UR5e+LEAP (80→27 shapes)
- Replace arm link collision meshes with properly-sized capsules
- Remove link_0 (base) and wrist_mount_link collisions
- Simplify finger collisions: remove link_0, extend link_1/link_2 toward base
- Replace fingertip OBJ meshes with capsule primitives
- Simplify palm: keep motor housings + main body + rear block + angled backing plate
- Delete thumb_link_1 collision, extend thumb_link_2 toward base
- Enable replace_cylinders_with_capsules and merge_fixed_joints in robot config

Co-Authored-By: Claude Opus 4.6 <noreply@anthropic.com>

File: source/isaaclab_tasks/isaaclab_tasks/manager_based/manipulation/y2r/assets/ur5e_leap/ur5e_leap_right_gemini305.urdf (robot description, URDF)
Before this commit: robot ur5e_leap_right, 40 links, 39 joints
Links:
- link index_link_0: geometry visual mesh filename=leap/meshes/visual/mcp_joint.obj
- link index_link_1: geometry collision box size=0.044 0.026 0.022; visual mesh filename=leap/meshes/visual/pip.obj
- link index_link_2: geometry collision box size=0.034 0.032 0.026; visual mesh filename=leap/meshes/visual/dip.obj
- link index_link_3: geometry collision cylinder length=0.02 radius=0.012; visual mesh filename=leap/meshes/visual/fingertip.obj
- link index_tip: geometry visual sphere radius=0.001
- link middle_link_0: geometry visual mesh filename=leap/meshes/visual/mcp_joint.obj
- link middle_link_1: geometry collision box size=0.044 0.026 0.022; visual mesh filename=leap/meshes/visual/pip.obj
- link middle_link_2: geometry collision box size=0.034 0.032 0.026; visual mesh filename=leap/meshes/visual/dip.obj
- link middle_link_3: geometry collision cylinder length=0.02 radius=0.012; visual mesh filename=leap/meshes/visual/fingertip.obj
- link middle_tip: geometry visual sphere radius=0.001
- link palm_frame: geometry visual sphere radius=0.001
- link palm_link: geometry collision box size=0.02 0.12 0.03; collision box size=0.022 0.026 0.034
- link ring_link_0: geometry visual mesh filename=leap/meshes/visual/mcp_joint.obj
- link ring_link_1: geometry collision box size=0.044 0.026 0.022; visual mesh filename=leap/meshes/visual/pip.obj
- link ring_link_2: geometry collision box size=0.034 0.032 0.026; visual mesh filename=leap/meshes/visual/dip.obj
- link ring_link_3: geometry collision cylinder length=0.02 radius=0.012; visual mesh filename=leap/meshes/visual/fingertip.obj
- link ring_tip: geometry visual sphere radius=0.001
- link thumb_link_1: geometry visual mesh filename=leap/meshes/visual/thumb_pip.obj
- link thumb_link_2: geometry collision box size=0.02 0.05 0.024; visual mesh filename=leap/meshes/visual/thumb_dip.obj
- link thumb_link_3: geometry collision box size=0.02 0.036 0.024; collision cylinder length=0.02 radius=0.012
- link thumb_tip: geometry visual sphere radius=0.001
- link ur5e_link_0: geometry visual mesh filename=ur5e/meshes/visual/base.obj
- link ur5e_link_1: geometry collision cylinder length=0.12 radius=0.06; visual mesh filename=ur5e/meshes/visual/shoulder.obj
- link ur5e_link_2: geometry collision cylinder length=0.45 radius=0.055; visual mesh filename=ur5e/meshes/visual/upperarm.obj
- link ur5e_link_3: geometry collision cylinder length=0.39 radius=0.045; visual mesh filename=ur5e/meshes/visual/forearm.obj
- link ur5e_link_4: geometry collision cylinder length=0.08 radius=0.04; visual mesh filename=ur5e/meshes/visual/wrist1.obj
- link ur5e_link_5: geometry collision cylinder length=0.07 radius=0.04; visual mesh filename=ur5e/meshes/visual/wrist2.obj
- link ur5e_link_6: geometry collision cylinder length=0.04 radius=0.035; visual mesh filename=ur5e/meshes/visual/wrist3.obj
- link wrist_mount_link: geometry visual mesh filename=wrist_mount.obj
Joints:
- joint hand_base_joint: axis (none) -> 0 0 1; limit (none) -> lower=0 upper=0 effort=0 velocity=0; type fixed -> revolute
- joint index_tip_joint: axis (none) -> 0 0 1; limit (none) -> lower=0 upper=0 effort=0 velocity=0; type fixed -> revolute
- joint middle_tip_joint: axis (none) -> 0 0 1; limit (none) -> lower=0 upper=0 effort=0 velocity=0; type fixed -> revolute
- joint palm_frame_joint: axis (none) -> 0 0 1; limit (none) -> lower=0 upper=0 effort=0 velocity=0; type fixed -> revolute
- joint ring_tip_joint: axis (none) -> 0 0 1; limit (none) -> lower=0 upper=0 effort=0 velocity=0; type fixed -> revolute
- joint thumb_tip_joint: axis (none) -> 0 0 1; limit (none) -> lower=0 upper=0 effort=0 velocity=0; type fixed -> revolute

Commit message: Add table penetration check for joint reset, palm frame offsets, tip offsets
Joint reset safety:
- Add reset_robot_joints_above_table() event that checks FK via
  update_articulations_kinematic() after writing randomized joints
- Envs where any hand body penetrates the table fall back to default
  arm+wrist positions (finger randomization preserved)
- Replace separate reset_robot_joints + reset_robot_wrist_joint events
  with single combined event
- Add wrist_joint_name, arm_joint_regex, hand_body_regex to robot config
  (single source of truth in YAML, no hardcoded defaults)

Palm frame & tip offsets:
- Add palm_frame_offset and tip_offsets to robot config
- Switch palm_body_name from palm_frame to palm_link (real body)
- Add get_palm_frame_pose_w() helper for computed palm frame
- Add hand_tips_state_with_offsets_b() observation term
- Simplify UR5E URDF (remove virtual palm_frame body, use fixed joint)

Config improvements:
- Add solver_position/velocity_iteration_count to simulation config
- Add PalmFrameOffsetConfig dataclass with Optional parsing support
- Update workspace x bounds [-0.85, -0.45]

Co-Authored-By: Claude Opus 4.6 <noreply@anthropic.com>

File: source/isaaclab_tasks/isaaclab_tasks/manager_based/manipulation/y2r/assets/ur5e_leap/ur5e_leap_right_gemini305.urdf (robot description, URDF)
Before this commit: robot ur5e_leap_right, 40 links, 39 joints
Links:
- link index_tip: geometry 
- link middle_tip: geometry 
- link palm_frame: geometry 
- link ring_tip: geometry 
- link thumb_tip: geometry 
- link ur5e_link_1: geometry visual mesh filename=ur5e/meshes/visual/shoulder.obj
Joints:
- joint index_tip_joint: axis 0 0 1 -> (none); limit lower=0 upper=0 effort=0 velocity=0 -> (none); type revolute -> fixed
- joint middle_tip_joint: axis 0 0 1 -> (none); limit lower=0 upper=0 effort=0 velocity=0 -> (none); type revolute -> fixed
- joint palm_frame_joint: axis 0 0 1 -> (none); limit lower=0 upper=0 effort=0 velocity=0 -> (none); type revolute -> fixed
- joint ring_tip_joint: axis 0 0 1 -> (none); limit lower=0 upper=0 effort=0 velocity=0 -> (none); type revolute -> fixed
- joint thumb_tip_joint: axis 0 0 1 -> (none); limit lower=0 upper=0 effort=0 velocity=0 -> (none); type revolute -> fixed

Commit message: Merge palm_link into ur5e_link_6, add abnormal_robot debug stats
URDF: hand_base_joint revolute→fixed so palm_link merges into ur5e_link_6
(removes phantom revolute joint with zero limits). Removed unused collision
geometry on one link. Regenerated USD asset.

Updated all palm_link references to ur5e_link_6 across env cfg, base.yaml,
and kuka_allegro.yaml. Recomputed palm_frame and camera offsets relative to
the new parent body.

Reward/curriculum tuning: num_envs 16384→20480, hand_pose_following weight
3.5→3.0, gate_floor [0.4,0.1]→[0.3,0.1], grasp_scale [0.4,0.0]→[0.9,0.1],
play difficulty initial 3→1.

Added config-gated abnormal_robot_state debug mode: accumulates per-joint
termination counts and prints a compact summary table every 1000 steps
instead of noisy per-step messages. Controlled by
terminations.abnormal_robot.debug in base.yaml.

Co-Authored-By: Claude Opus 4.6 <noreply@anthropic.com>

File: source/isaaclab_tasks/isaaclab_tasks/manager_based/manipulation/y2r/assets/ur5e_leap/ur5e_leap_right_gemini305.urdf (robot description, URDF)
Before this commit: robot ur5e_leap_right, 40 links, 39 joints
Links:
- link thumb_link_0: geometry visual mesh filename=leap/meshes/visual/pip.obj
Joints:
- joint hand_base_joint: axis 0 0 1 -> (none); limit lower=0 upper=0 effort=0 velocity=0 -> (none); type revolute -> fixed

Commit message: New fingertip STL, link_2 contact sensors, collision tuning, config improvements
URDF:
- Replace fingertip visuals with new finger_tip.stl + chopped connector OBJs
- Decompose fingertip collisions into base box + square block + angled capsule
- Shorten finger link_1 and thumb link_2 collision boxes from palm side
- Add thumb connector collision box from original geometry
- Increase link masses/inertias for stability

Rewards:
- Add cached _get_finger_contact_mags() using max(link_3, link_2) per finger
- Replace 3 duplicated contact sensor reads with single cached call
- Replace hard contact gate in finger_manipulation with soft contact_factor
- Add contact gating params to finger_manipulation reward

Env config:
- Add link_2 contact sensors for all 4 fingers (ur5e_leap)
- Add velocity_limit_sim to UR5e+LEAP actuator config
- Support abnormal_robot.enabled flag to disable termination
- Support null object_x/object_y to inherit workspace bounds
- Filter early_termination term_keys for disabled terminations

Other:
- Add per-joint keyboard control mode (Up/Down to cycle, J/K to move)
- Tune curriculum, friction, termination thresholds in base.yaml

Co-Authored-By: Claude Opus 4.6 <noreply@anthropic.com>

File: source/isaaclab_tasks/isaaclab_tasks/manager_based/manipulation/y2r/assets/ur5e_leap/ur5e_leap_right_gemini305.urdf (robot description, URDF)
Before this commit: robot ur5e_leap_right, 40 links, 39 joints
Links:
- link index_link_0: mass 0.044 -> 0.1
- link index_link_1: mass 0.032 -> 0.1; geometry collision box size=0.034 0.026 0.022; visual mesh filename=leap/meshes/visual/pip.obj
- link index_link_2: mass 0.037 -> 0.1
- link index_link_3: mass 0.016 -> 0.06; geometry collision box size=0.019 0.008 0.033; collision box size=0.019 0.018 0.019
- link middle_link_0: mass 0.044 -> 0.1
- link middle_link_1: mass 0.032 -> 0.1; geometry collision box size=0.034 0.026 0.022; visual mesh filename=leap/meshes/visual/pip.obj
- link middle_link_2: mass 0.037 -> 0.1
- link middle_link_3: mass 0.016 -> 0.06; geometry collision box size=0.019 0.008 0.033; collision box size=0.019 0.018 0.019
- link ring_link_0: mass 0.044 -> 0.1
- link ring_link_1: mass 0.032 -> 0.1; geometry collision box size=0.034 0.026 0.022; visual mesh filename=leap/meshes/visual/pip.obj
- link ring_link_2: mass 0.037 -> 0.1
- link ring_link_3: mass 0.016 -> 0.06; geometry collision box size=0.019 0.008 0.033; collision box size=0.019 0.018 0.019
- link thumb_link_0: mass 0.032 -> 0.1
- link thumb_link_1: mass 0.003 -> 0.1
- link thumb_link_2: mass 0.038 -> 0.1; geometry collision box size=0.02 0.04 0.024; visual mesh filename=leap/meshes/visual/thumb_dip.obj
- link thumb_link_3: mass 0.049 -> 0.1; geometry collision box size=0.019 0.008 0.033; collision box size=0.019 0.018 0.019

Commit message: Tighten LEAP hand finger spread joint limits, disable student mode in play config
- Reduce index/middle/ring _joint_0 (abduction) limits from ±1.047 rad (±60°)
  to ±0.595 rad (±34°), matching Allegro hand spec
- Regenerated USD asset from updated URDF
- play.yaml: set use_student_mode to false, disable student visualization
  markers and camera debug viewer

Co-Authored-By: Claude Opus 4.6 <noreply@anthropic.com>

File: source/isaaclab_tasks/isaaclab_tasks/manager_based/manipulation/y2r/assets/ur5e_leap/ur5e_leap_right_gemini305.urdf (robot description, URDF)
Before this commit: robot ur5e_leap_right, 40 links, 39 joints
Joints:
- joint index_joint_0: limit lower=-1.047 upper=1.047 effort=0.5 velocity=8.48 -> lower=-0.595 upper=0.595 effort=0.5 velocity=8.48
- joint middle_joint_0: limit lower=-1.047 upper=1.047 effort=0.5 velocity=8.48 -> lower=-0.595 upper=0.595 effort=0.5 velocity=8.48
- joint ring_joint_0: limit lower=-1.047 upper=1.047 effort=0.5 velocity=8.48 -> lower=-0.595 upper=0.595 effort=0.5 velocity=8.48

Commit message: SAPG support, network extra_param type, flash attention toggle, sim tuning
- Add SAPG config blocks to all y2r agent configs and update fixed_sigma
  from bool to string enum ('fixed'/'coef_cond'/'obs_cond') across all
  rl_games configs in IsaacLab
- Networks (point_transformer, pointnet_tnet): add extra_param net type
  with learnable coefficient embeddings, coef_cond sigma, flash_attention
  toggle (math backend for batch > 65535), _prepare_obs() for obs
  rearrangement
- Point transformer MLP widened to [1024, 1024, 512, 512], minibatch 61440
- Sim: num_envs 61440, abnormal_robot enabled, curriculum step_interval
  30000, gpu_max_rigid_patch_count ~2M
- Compat: pbt.py process_infos **kwargs, distill_agent unpack _intr_rewards,
  train.py force FP32 for SAPG mixed_expl
- URDF/asset hash updates for ur5e_leap

Co-Authored-By: Claude Opus 4.6 <noreply@anthropic.com>

File: source/isaaclab_tasks/isaaclab_tasks/manager_based/manipulation/y2r/assets/ur5e_leap/ur5e_leap_right_gemini305.urdf (robot description, URDF)
Before this commit: robot ur5e_leap_right, 40 links, 39 joints
Joints:
- joint index_joint_0: limit lower=-0.595 upper=0.595 effort=0.5 velocity=8.48 -> lower=-0.349 upper=0.349 effort=0.5 velocity=8.48
- joint middle_joint_0: limit lower=-0.595 upper=0.595 effort=0.5 velocity=8.48 -> lower=-0.349 upper=0.349 effort=0.5 velocity=8.48
- joint ring_joint_0: limit lower=-0.595 upper=0.595 effort=0.5 velocity=8.48 -> lower=-0.349 upper=0.349 effort=0.5 velocity=8.48

Commit message: SysID infrastructure: sysid config layer, fitting script, URDF effort limits
Add sysid mode for config_loader, sysid.yaml config layer, and
sysid_fit_isaac.py CMA-ES fitting script. Update URDF effort limits
and USD asset config for ur5e_leap.

Co-Authored-By: Claude Opus 4.6 (1M context) <noreply@anthropic.com>

File: source/isaaclab_tasks/isaaclab_tasks/manager_based/manipulation/y2r/assets/ur5e_leap/ur5e_leap_right_gemini305.urdf (robot description, URDF)
Before this commit: robot ur5e_leap_right, 40 links, 39 joints
Links:
- link index_link_0: mass 0.1 -> 0.044
- link index_link_1: mass 0.1 -> 0.032
- link index_link_2: mass 0.1 -> 0.037
- link index_link_3: mass 0.06 -> 0.016
- link middle_link_0: mass 0.1 -> 0.044
- link middle_link_1: mass 0.1 -> 0.032
- link middle_link_2: mass 0.1 -> 0.037
- link middle_link_3: mass 0.06 -> 0.016
- link ring_link_0: mass 0.1 -> 0.044
- link ring_link_1: mass 0.1 -> 0.032
- link ring_link_2: mass 0.1 -> 0.037
- link ring_link_3: mass 0.06 -> 0.016
- link thumb_link_0: mass 0.1 -> 0.032
- link thumb_link_1: mass 0.1 -> 0.003
- link thumb_link_2: mass 0.1 -> 0.038
- link thumb_link_3: mass 0.1 -> 0.049

Commit message: Widen finger abduction limits to ±40°; tweak env config
- index/middle/ring joint_0 limits: ±0.349 → ±0.6981 rad (±20° → ±40°)
- object_pc history: 1 → 4
- action_l2 finger_scale: 0.06 → 0.05
- Refresh procedural and ur5e_leap_usd asset hashes

Co-Authored-By: Claude Opus 4.7 (1M context) <noreply@anthropic.com>

File: source/isaaclab_tasks/isaaclab_tasks/manager_based/manipulation/y2r/assets/ur5e_leap/ur5e_leap_right_gemini305.urdf (robot description, URDF)
Before this commit: robot ur5e_leap_right, 40 links, 39 joints
Joints:
- joint index_joint_0: limit lower=-0.349 upper=0.349 effort=0.5 velocity=8.48 -> lower=-0.6981 upper=0.6981 effort=0.5 velocity=8.48
- joint middle_joint_0: limit lower=-0.349 upper=0.349 effort=0.5 velocity=8.48 -> lower=-0.6981 upper=0.6981 effort=0.5 velocity=8.48
- joint ring_joint_0: limit lower=-0.349 upper=0.349 effort=0.5 velocity=8.48 -> lower=-0.6981 upper=0.6981 effort=0.5 velocity=8.48

Commit message: Tune contact factor + terminations + heads + URDF; cylinder pose-axis viz
- Contact factor restructured: palm folded into the gate (gate_input =
  1.0·thumb_sat + 0.25·palm_sat, max 1.25 unclipped), Tier 2 additive
  bonus removed. palm_threshold/palm_ramp retained for the palm side.
- Teacher PT num_heads 8 → 4 (head_dim 64/4 = 16); student PT 16 → 8
  (head_dim 128/8 = 16).
- Terminations: trajectory_deviation pos [0.2, 0.1] → [0.15, 0.1], rot
  [2.0, 1.0] → [1.5, 1.0]. hand_pose_deviation pos [0.175, 0.075] →
  [0.2, 0.1], rot [2.0, 0.9] → [2.0, 1.0]. Tighter object cap, looser
  palm cap so the policy can deviate the palm while keeping object on
  track.
- Trajectory: explore.max_rotation 1.0 → 1.5708 (90°). Keypoints
  roll_perturbation 0.3 → 0.0 (disabled).
- URDF abduction limits ±40° → ±25° on index/middle/ring joint_0
  (thumb untouched).
- Pose-axis viz: replaced arrow_x.usd prim with three thin cylinders
  (red/green/blue), 5 mm shaft, length 10/12 cm, offset by length/2 so
  the proximal end sits at the frame origin. Decouples thickness from
  length and makes axes visible to offscreen RecordVideo cameras.

Co-Authored-By: Claude Opus 4.7 (1M context) <noreply@anthropic.com>

File: source/isaaclab_tasks/isaaclab_tasks/manager_based/manipulation/y2r/assets/ur5e_leap/ur5e_leap_right_gemini305.urdf (robot description, URDF)
Before this commit: robot ur5e_leap_right, 40 links, 39 joints
Joints:
- joint index_joint_0: limit lower=-0.6981 upper=0.6981 effort=0.5 velocity=8.48 -> lower=-0.4363 upper=0.4363 effort=0.5 velocity=8.48
- joint middle_joint_0: limit lower=-0.6981 upper=0.6981 effort=0.5 velocity=8.48 -> lower=-0.4363 upper=0.4363 effort=0.5 velocity=8.48
- joint ring_joint_0: limit lower=-0.6981 upper=0.6981 effort=0.5 velocity=8.48 -> lower=-0.4363 upper=0.4363 effort=0.5 velocity=8.48
