Commit message: Update UR5e WSG50 visual calibration assets

File: source/isaaclab_tasks/isaaclab_tasks/manager_based/manipulation/y2r/assets/ur5e_gemini_wsg50/ur5e_gemini_wsg50.urdf (robot description, URDF)
Before this commit: robot ur5e_gemini_wsg50, 26 links, 25 joints
Links:
- added link finger_holder_left_visual_link, mass 0.001; visual mesh filename=external_meshes/finger_holder_left.obj
- added link finger_holder_right_visual_link, mass 0.001; visual mesh filename=external_meshes/finger_holder_right.obj
- added link wsg_mount_visual_link, mass 0.001; visual mesh filename=external_meshes/wsg50_mount.stl
Joints:
- added joint finger_holder_left_visual_joint: type fixed, parent soft_finger_left_link, child finger_holder_left_visual_link, origin xyz=-0.001 0.101 0.013 rpy=1.570796327 0 0
- added joint finger_holder_right_visual_joint: type fixed, parent soft_finger_right_link, child finger_holder_right_visual_link, origin xyz=0.001 0.1 0.013 rpy=1.570796327 0 0
- added joint wsg_mount_visual_joint: type fixed, parent wsg_base_link, child wsg_mount_visual_link, origin xyz=0 0 0 rpy=0 0 0
