Commit message: Update WSG palm frame calibration
Set the WSG palm frame yaw to match the adjusted gripper pose and add a WSG teacher finetune task layer that keeps tight hand-pose termination while inheriting base reward and object-deviation settings.

Co-Authored-By: OpenAI Codex <noreply@openai.com>

File: source/isaaclab_tasks/isaaclab_tasks/manager_based/manipulation/y2r/assets/ur5e_gemini_wsg50/ur5e_gemini_wsg50.urdf (robot description, URDF)
Before this commit: robot ur5e_gemini_wsg50, 29 links, 28 joints
Joints:
- joint palm_frame_joint: origin xyz=0 0 0.146 rpy=0 0 0 -> xyz=0 0 0.146 rpy=0 0 1.570796327
